File: hw/EspFanControl.kicad_pcb (KiCad board)
At the start: 2 copper layers, 40.3 x 18 mm, 21 parts, among them J1 DSP, J2 FAN, J3 IFC, J4 O-Wire, J5 5V, Q1 BC847, Q2 AO3401A, SW1 RST, SW2 PGM, U1 ESP-12F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

Commit message: update: cleanup
Connections:
- U1 pad 19: /SCL -> /SDA
- U1 pad 20: /SDA -> /SCL
Routing:
- net /SDA: track 39.9 -> 37.3 mm, vias 1 -> 2
- net /SCL: track 36.2 -> 38.9 mm, vias 2 -> 1
- net GND: vias 26 -> 27
