File: hw/EspFanControl.kicad_sch (KiCad schematic)
At the start: 21 parts, among them J1 DSP, J2 FAN, J3 IFC, J4 O-Wire, J5 5V, Q1 BC847, Q2 AO3401A, SW1 RST, SW2 PGM, U1 ESP-12F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

Commit message: update: cleanup
Connections:
- net SCL: now also U1.20 (GPIO5); no longer U1.19 (GPIO4)
- net SDA: now also U1.19 (GPIO4); no longer U1.20 (GPIO5)
Changed lines of the file:
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@@
     (effects (font (size 1.27 1.27)) (justify left bottom))
   )
-  (label "SCL" (at 62.23 81.28 0)
+  (label "SCL" (at 62.23 83.82 0)
     (effects (font (size 1.27 1.27)) (justify left bottom))
   )
@@
     (effects (font (size 1.27 1.27)) (justify right bottom))
   )
-  (label "SDA" (at 62.23 83.82 0)
+  (label "SDA" (at 62.23 81.28 0)
     (effects (font (size 1.27 1.27)) (justify left bottom))
   )

Commit message: add
Other:
- note added: "Buttons"
- note added: "DS18B20"
- note added: "ESP8266"
- note added: "FAN"
- note added: "Fan-Ctrl"
- note added: "OLED"
- note added: "PGM"
- note added: "POWER"
- note added: "Pull-Up/Down"
- note added: "Supply"
- moved on the sheet: C1, D1, J1, J2, J3, J4, J5, Q1, Q2, R1, R2, R3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
